File: Copy of Parcial_1.brd (EAGLE design)
At the start: 68.6 x 53.3 mm, 83 parts

Commit message: Se controlan filas y columnas independientemente
Parts:
- removed D1, D8: (no value), AUTODESK_CIRCUITS_BREADBOARD:LED5MM
- added D65, D66: (no value), AUTODESK_CIRCUITS_BREADBOARD:LED-RGB-THRU
- D10, D11, D12, D13, D14, D15, D16, D17, D18, D19, D2, D20, D21, D22, D23, D24, D25, D26, D27, D28, D29, D3, D30, D31, D32, D33, D34, D35, D36, D37, D38, D39, D4, D40, D41, D42, D43, D44, D45, D46, D47, D48, D49, D5, D50, D51, D52, D53, D54, D55, D56, D57, D58, D59, D6, D60, D61, D62, D63, D64, D7, D9: device AUTODESK_CIRCUITS_BREADBOARD:LED5MM -> AUTODESK_CIRCUITS_BREADBOARD:LED-RGB-THRU
- R1, R10, R11, R12, R13, R14, R15, R16, R2, R3, R4, R5, R6, R7, R8, R9: value 560‎Ω -> 220‎Ω
- moved R15 838.2 mm to (5.00, 200.6)
- moved R16 838.2 mm to (5.00, 213.3)
- moved R10 825.5 mm to (5.00, 149.8)
- moved R11 825.5 mm to (5.00, 162.5)
- moved R12 825.5 mm to (5.00, 175.2)
- moved R13 825.5 mm to (5.00, 187.9)
- moved R1 825.5 mm to (5.00, 137.1)
- moved R4 825.5 mm to (5.00, 124.4)
- moved R3 825.5 mm to (5.00, 111.7)
- moved R8 825.5 mm to (5.00, 86.3)
- moved R9 825.5 mm to (5.00, 99.0)
- moved R2 812.8 mm to (5.00, 48.2)
- moved R5 812.8 mm to (5.00, 60.9)
- moved R6 812.8 mm to (5.00, 73.6)
- moved D14 685.8 mm to (5.00, 899.1)
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Connections:
- removed net N$1 (its old number): R16.2, U4.1
- removed net N$11 (its old number): R4.2, U3.2
- removed net N$14 (its old number): R5.2, U3.3
- removed net N$17 (its old number): R2.2, U3.15
- removed net N$8 (its old number): R6.2, U3.4
- new net N$19: R14.1, U4.3
- new net N$32: D59.3, D60.3, D61.3, D62.3, D63.3, D64.3, D65.3, D66.3, R10.1
- new net N$35: D10.3, D11.3, D12.3, D13.3, D14.3, D15.3, D16.3, D9.3, R1.1
- new net N$4: R5.2, U3.4
- new net N$6: R2.2, U3.7
- net N$10: now also R6.2, U3.3; no longer R9.2, U3.7
- net N$13: now also R9.2, U3.15; no longer R7.2, U3.5
- net N$20: now also D19.2, D2.2, D27.2, D35.2, D43.2, D51.2, D59.2, D9.2; no longer D1.K, D17.K, D25.K, D33.K, D41.K, D49.K, D57.K, D9.K
- net N$21: now also D10.2, D20.2, D28.2, D3.2, D36.2, D44.2, D52.2, D60.2; no longer D10.K, D18.K, D2.K, D26.K, D34.K, D42.K, D50.K, D58.K
- net N$22: now also D11.2, D21.2, D29.2, D37.2, D4.2, D45.2, D53.2, D61.2; no longer D11.K, D19.K, D27.K, D3.K, D35.K, D43.K, D51.K, D59.K
- net N$23: now also D12.2, D22.2, D30.2, D38.2, D46.2, D5.2, D54.2, D62.2; no longer D12.K, D20.K, D28.K, D36.K, D4.K, D44.K, D52.K, D60.K
- net N$24: now also D13.2, D23.2, D31.2, D39.2, D47.2, D55.2, D6.2, D63.2; no longer D13.K, D21.K, D29.K, D37.K, D45.K, D5.K, D53.K, D61.K
- net N$25: now also D14.2, D24.2, D32.2, D40.2, D48.2, D56.2, D64.2, D7.2; no longer D14.K, D22.K, D30.K, D38.K, D46.K, D54.K, D6.K, D62.K
- net N$26: now also D15.2, D17.2, D25.2, D33.2, D41.2, D49.2, D57.2, D65.2; no longer D15.K, D23.K, D31.K, D39.K, D47.K, D55.K, D63.K, D7.K
- net N$27: now also D16.2, D18.2, D26.2, D34.2, D42.2, D50.2, D58.2, D66.2; no longer D16.K, D24.K, D32.K, D40.K, D48.K, D56.K, D64.K, D8.K
- net N$28: now also D51.3, D52.3, D53.3, D54.3, D55.3, D56.3, D57.3, D58.3, R13.1; no longer D1.A, D2.A, D3.A, D4.A, D5.A, D6.A, D7.A, D8.A, R1.1
- net N$29: now also D27.3, D28.3, D29.3, D30.3, D31.3, D32.3, D33.3, D34.3, R14.2; no longer D10.A, D11.A, D12.A, D13.A, D14.A, D15.A, D16.A, D9.A, R10.1
- net N$3: now also R8.2, U3.1; no longer R15.2, U4.2
- net N$30: now also D17.3, D18.3, D2.3, D3.3, D4.3, D5.3, D6.3, D7.3; no longer D17.A, D18.A, D19.A, D20.A, D21.A, D22.A, D23.A, D24.A
- net N$31: now also D19.3, D20.3, D21.3, D22.3, D23.3, D24.3, D25.3, D26.3; no longer D25.A, D26.A, D27.A, D28.A, D29.A, D30.A, D31.A, D32.A
- net N$36: now also R16.1, U4.1; no longer D57.A, D58.A, D59.A, D60.A, D61.A, D62.A, D63.A, D64.A, R13.1
- net N$37: now also R15.1, U4.2; no longer D33.A, D34.A, D35.A, D36.A, D37.A, D38.A, D39.A, D40.A, R14.1
- net N$38: now also D35.3, D36.3, D37.3, D38.3, D39.3, D40.3, D41.3, D42.3, R15.2; no longer D41.A, D42.A, D43.A, D44.A, D45.A, D46.A, D47.A, D48.A, R15.1
- net N$39: now also D43.3, D44.3, D45.3, D46.3, D47.3, D48.3, D49.3, D50.3, R16.2; no longer D49.A, D50.A, D51.A, D52.A, D53.A, D54.A, D55.A, D56.A, R16.1
- net N$5: now also R3.2, U3.6; no longer R14.2, U4.3
- net N$7: now also R7.2, U3.2; no longer R3.2, U3.1
- net N$9: now also R4.2, U3.5; no longer R8.2, U3.6
