File: Copy of Copy of Parcial_1.brd (EAGLE design)
At the start: 68.6 x 53.3 mm, 83 parts

Commit message: Se decide seguir con la funcion shiftOut, pero se esta analizando su funcionamiento realizando pruebas
Parts:
- removed R2, R3, R4, R5, R6, R7, R8, R9: 220‎Ω, AUTODESK_CIRCUITS_BREADBOARD:0207/10
- moved D10 88.9 mm to (5.00, 759.4)
- moved D11 88.9 mm to (5.00, 772.1)
- moved D12 88.9 mm to (5.00, 784.8)
- moved D13 88.9 mm to (5.00, 797.5)
- moved D14 88.9 mm to (5.00, 810.2)
- moved D15 88.9 mm to (5.00, 822.9)
- moved D16 88.9 mm to (5.00, 835.6)
- moved D41 88.9 mm to (5.00, 518.1)
- moved D42 88.9 mm to (5.00, 530.8)
- moved D43 88.9 mm to (5.00, 543.5)
- moved D44 88.9 mm to (5.00, 556.2)
- moved D45 88.9 mm to (5.00, 568.9)
- moved D46 88.9 mm to (5.00, 581.6)
- moved D47 88.9 mm to (5.00, 594.3)
- moved D48 88.9 mm to (5.00, 607.0)
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Connections:
- removed net N$20 (its old number): D19.2, D2.2, D27.2, D35.2, D43.2, D51.2, D59.2, D9.2, R2.1
- removed net N$21 (its old number): D10.2, D20.2, D28.2, D3.2, D36.2, D44.2, D52.2, D60.2, R3.1
- removed net N$22 (its old number): D11.2, D21.2, D29.2, D37.2, D4.2, D45.2, D53.2, D61.2, R4.1
- removed net N$23 (its old number): D12.2, D22.2, D30.2, D38.2, D46.2, D5.2, D54.2, D62.2, R5.1
- removed net N$24 (its old number): D13.2, D23.2, D31.2, D39.2, D47.2, D55.2, D6.2, D63.2, R6.1
- removed net N$25 (its old number): D14.2, D24.2, D32.2, D40.2, D48.2, D56.2, D64.2, D7.2, R7.1
- removed net N$26 (its old number): D15.2, D17.2, D25.2, D33.2, D41.2, D49.2, D57.2, D65.2, R8.1
- removed net N$27 (its old number): D16.2, D18.2, D26.2, D34.2, D42.2, D50.2, D58.2, D66.2, R9.1
- net N$10: now also D13.2, D23.2, D31.2, D39.2, D47.2, D55.2, D6.2, D63.2; no longer R6.2
- net N$12: now also U1.4; no longer U1.12
- net N$13: now also D16.2, D18.2, D26.2, D34.2, D42.2, D50.2, D58.2, D66.2; no longer R9.2
- net N$14: now also U1.3; no longer U1.11
- net N$3: now also D15.2, D17.2, D25.2, D33.2, D41.2, D49.2, D57.2, D65.2; no longer R8.2
- net N$4: now also D12.2, D22.2, D30.2, D38.2, D46.2, D5.2, D54.2, D62.2; no longer R5.2
- net N$5: now also D10.2, D20.2, D28.2, D3.2, D36.2, D44.2, D52.2, D60.2; no longer R3.2
- net N$6: now also D19.2, D2.2, D27.2, D35.2, D43.2, D51.2, D59.2, D9.2; no longer R2.2
- net N$7: now also D14.2, D24.2, D32.2, D40.2, D48.2, D56.2, D64.2, D7.2; no longer R7.2
- net N$8: now also U1.2; no longer U1.8
- net N$9: now also D11.2, D21.2, D29.2, D37.2, D4.2, D45.2, D53.2, D61.2; no longer R4.2
